Commit message: updated the yaml files and xacro files to rotate the robot 90 degrees

File: xarm_description/urdf/gripper/xarm_gripper.urdf.xacro (robot description, xacro)
@@ -9,4 +9,5 @@
       </joint>
     </xacro:unless>
+    <!-- THIS ONE SEEMS TO WORK OKAY -->
     <link name="${prefix}xarm_gripper_base_link">
       <inertial>

File: xarm_description/urdf/xarm7/xarm7.urdf.xacro (robot description, xacro)
@@ -40,5 +40,5 @@
     <link name="${prefix}link_base">
       <inertial>
-        <origin xyz="-0.021131 -0.0016302 0.056488" rpy="0 0 0" />
+        <origin xyz="-0.021131 -0.0016302 0.056488" rpy="0 0 ${-3.14159265/2}" />
         <mass value="0.88556" />
         <inertia
@@ -49,10 +49,10 @@
         mesh_filename="xarm7/visual/link_base"
         origin_xyz="0 0 0"
-        origin_rpy="0 0 0"
+        origin_rpy="0 0 ${-3.14159265/2}"
         material_name="${prefix}White" />
       <xacro:common_link_collision
         mesh_filename="xarm7/visual/link_base"
         origin_xyz="0 0 0"
-        origin_rpy="0 0 0" />
+        origin_rpy="0 0 ${-3.14159265/2}" />
     </link>
     <link name="${prefix}link1">
